Commit message: fixed visual bugs of robot model; aesthetic matters!

File: RoboRTS_Gazebo/robots/infantry.urdf.xacro (robot description, xacro)
@@ -34,14 +34,14 @@
     <collision>
     <origin
-        xyz="-0.1 0 0.2"
+        xyz="-0.1 0 0.15"
         rpy="0 0 0" />
     <geometry>
       <box
-        size= "0.2 0.1 0.25"/>
-      </geometry>
-    </collision>
-    <visual>
-      <origin
-        xyz="0 0 0.05"
+        size= "0.2 0.1 0.3"/>
+      </geometry>
+    </collision>
+    <visual>
+      <origin
+        xyz="0 0 0"
         rpy="0 0 0" />
       <geometry>
@@ -118,9 +118,9 @@
           filename="package://roborts_gazebo/meshes/br_wheel_link.STL" />
       </geometry>
-      <material
+      <!-- <material
         name="roborts_red">
         <color
           rgba="${242/255} ${38/255} ${19/255} 1" />
-      </material>
+      </material> -->
     </visual>
     <collision>
@@ -175,5 +175,5 @@
       <origin
         xyz="0 0 0"
-        rpy="0 0 0" />
+        rpy="0 0 3.1416" />
       <geometry>
         <mesh
@@ -237,5 +237,5 @@
       <origin
         xyz="0 0 0"
-        rpy="0 0 0" />
+        rpy="0 0 3.1416" />
       <geometry>
         <mesh
@@ -503,5 +503,5 @@
   <joint
     name="pitch_link_to_camera_wheel_joint"
-    type="fixed">
+    type="fixed">collision
     <origin
       xyz="0.041 0 0.049"
@@ -558,5 +558,5 @@
     type="fixed">
     <origin
-      xyz="0 0 0.1"
+      xyz="0 0 0.15"
       rpy="0 0 0" />
     <parent
