Commit message: changed collision box for the robots so that laser can detect other robots

File: RoboRTS_Gazebo/robots/infantry.gazebo.xacro (robot description, xacro)
@@ -3,4 +3,5 @@
 	name="infantry_xacro">
   <xacro:arg name="namespace_xacro" default=""/>
+  <xacro:arg name="visualize" default="false"/>
   <gazebo reference="fr_wheel_link">
     <material>Gazebo/White</material>
@@ -34,4 +35,5 @@
   <gazebo reference="base_link">
     <material>Gazebo/Black</material>
+    <laserRetro>700</laserRetro>
     <turnGravityOff>false</turnGravityOff>
     <!--<kinematic>1</kinematic>-->
@@ -42,5 +44,5 @@
   </gazebo> -->
   <gazebo reference="base_laser_link">
-    <material>Gazebo/Black</material>
+    <material>Gazebo/Gold</material>
     <turnGravityOff>false</turnGravityOff>
   </gazebo>
@@ -49,5 +51,6 @@
     <sensor type="ray" name="head_hokuyo_sensor">
       <pose>0 0 0.2 0 0 0</pose>
-      <visualize>false</visualize>
+      <!-- original value 0 0 0.2 0 0 0  -->
+      <visualize>$(arg visualize)</visualize>
       <update_rate>15</update_rate>
       <ray>

File: RoboRTS_Gazebo/robots/infantry.urdf.xacro (robot description, xacro)
@@ -21,17 +21,37 @@
     izz="0.32438" />
     </inertial>
-    <collision>
-    <origin
-    xyz="0 0 0"
-    rpy="0 0 0" />
+    <!-- base box -->
+    <collision>
+    <origin
+        xyz="0 0 0"
+        rpy="0 0 0" />
     <geometry>
-    <box
-    size= "0.55 0.4 0.1"
-    />
-    </geometry>
-    </collision>
-    <visual>
-      <origin
-        xyz="0 0 0"
+      <box
+        size= "0.55 0.4 0.1"/>
+      </geometry>
+    </collision>
+    <!-- short stick of the cross-->
+    <collision>
+    <origin
+        xyz="0 0 0.05"
+        rpy="0 0 0" />
+    <geometry>
+      <box
+        size= "0.1 0.4 0.15"/>
+      </geometry>
+    </collision>
+    <!-- long stick of the cross-->
+    <collision>
+    <origin
+        xyz="0 0 0.05"
+        rpy="0 0 0" />
+    <geometry>
+      <box
+        size= "0.55 0.1 0.15"/>
+      </geometry>
+    </collision>
+    <visual>
+      <origin
+        xyz="0 0 0.05"
         rpy="0 0 0" />
       <geometry>
@@ -582,7 +602,4 @@
         />
       </geometry>
-      <material
-        name="">
-        <color
           rgba="0.75294 0.75294 0.75294 1" />
       </material>

Commit message: improved collision box of base link

File: RoboRTS_Gazebo/robots/infantry.gazebo.xacro (robot description, xacro)
@@ -57,13 +57,13 @@
         <scan>
           <horizontal>
-            <samples>720</samples>
+            <samples>270</samples>
             <resolution>0.5</resolution>
-            <min_angle>-3.14159</min_angle>
-            <max_angle>3.14159</max_angle>
+            <min_angle>-2.35619</min_angle>
+            <max_angle>2.35619</max_angle>
           </horizontal>
         </scan>
         <range>
-          <min>0.3</min>
-          <max>4.5</max>
+          <min>0.15</min>
+          <max>8.0</max>
           <resolution>0.3</resolution>
         </range>

File: RoboRTS_Gazebo/robots/infantry.urdf.xacro (robot description, xacro)
@@ -31,22 +31,12 @@
       </geometry>
     </collision>
-    <!-- short stick of the cross-->
-    <collision>
-    <origin
-        xyz="0 0 0.05"
+    <!-- collision box behind laser -->
+    <collision>
+    <origin
+        xyz="-0.1 0 0.2"
         rpy="0 0 0" />
     <geometry>
       <box
-        size= "0.1 0.4 0.15"/>
-      </geometry>
-    </collision>
-    <!-- long stick of the cross-->
-    <collision>
-    <origin
-        xyz="0 0 0.05"
-        rpy="0 0 0" />
-    <geometry>
-      <box
-        size= "0.55 0.1 0.15"/>
+        size= "0.2 0.1 0.25"/>
       </geometry>
     </collision>

Commit message: added led light

File: RoboRTS_Gazebo/robots/infantry.gazebo.xacro (robot description, xacro)
@@ -4,4 +4,13 @@
   <xacro:arg name="namespace_xacro" default=""/>
   <xacro:arg name="visualize" default="false"/>
+  <xacro:arg name="led_color" default="Red"/>
+  <gazebo reference="led_Link">
+    <material>Gazebo/$(arg led_color)</material>
+    <turnGravityOff>false</turnGravityOff>
+  </gazebo>
+  <gazebo reference="armor_link">
+    <material>Gazebo/Black</material>
+    <turnGravityOff>false</turnGravityOff>
+  </gazebo>
   <gazebo reference="fr_wheel_link">
     <material>Gazebo/White</material>

File: RoboRTS_Gazebo/robots/infantry.urdf.xacro (robot description, xacro)
@@ -118,9 +118,9 @@
           filename="package://roborts_gazebo/meshes/br_wheel_link.STL" />
       </geometry>
-      <!-- <material
-        name="roborts_red">
-        <color
-          rgba="${242/255} ${38/255} ${19/255} 1" />
-      </material> -->
+      <material
+        name="">
+        <color
+          rgba="0.79216 0.81961 0.93333 1" />
+      </material>
     </visual>
     <collision>
@@ -663,3 +663,47 @@
       xyz="0 0 0" />
   </joint>
+<link
+    name="led_Link">
+    <inertial>
+      <origin
+        xyz="-0.27282 -0.063339 0.010089"
+        rpy="0 0 0" />
+      <mass
+        value="0.028183" />
+      <inertia
+        ixx="0.00037048"
+        ixy="7.803E-06"
+        ixz="9.4378E-05"
+        iyy="0.0011379"
+        iyz="-1.4266E-06"
+        izz="0.0014674" />
+    </inertial>
+    <visual>
+      <origin
+        xyz="0.28244 0.063339 0.061918"
+        rpy="0 0 0" />
+      <geometry>
+        <mesh
+          filename="package://roborts_gazebo/meshes/led_link.STL" />
+      </geometry>
+      <!-- <material
+        name="">
+        <color
+          rgba="1 0 0 1" />
+      </material> -->
+    </visual>
+  </link>
+  <joint
+    name="base_link_to_led_joint"
+    type="fixed">
+    <origin
+      xyz="0 0 0"
+      rpy="0 0 0" />
+    <parent
+      link="base_link" />
+    <child
+      link="led_Link" />
+    <axis
+      xyz="0 0 0" />
+  </joint>
 </robot>

File: RoboRTS_Gazebo/robots/infantry_blue.xacro (robot description, xacro)
@@ -4,3 +4,4 @@
         <xacro:include filename="$(find roborts_gazebo)/robots/infantry.gazebo.xacro" />
         <!--<xacro:include filename="$(find roborts_gazebo)/robots/infantry.transmission.xacro" />-->
+        <xacro:led_color name="Blue"/>
 </robot>

File: RoboRTS_Gazebo/robots/infantry_red.xacro (robot description, xacro)
@@ -4,3 +4,4 @@
         <xacro:include filename="$(find roborts_gazebo)/robots/infantry.gazebo.xacro" />
         <!--<xacro:include filename="$(find roborts_gazebo)/robots/infantry.transmission.xacro" />-->
+        <xacro:led_color name="Red"/>
 </robot>

Commit message: Added four armors and fixed the led issue

File: RoboRTS_Gazebo/robots/infantry.gazebo.xacro (robot description, xacro)
@@ -7,4 +7,20 @@
   <gazebo reference="led_Link">
     <material>Gazebo/$(arg led_color)</material>
+    <turnGravityOff>false</turnGravityOff>
+  </gazebo>
+  <gazebo reference="right_armor_link">
+    <material>Gazebo/White</material>
+    <turnGravityOff>false</turnGravityOff>
+  </gazebo>
+  <gazebo reference="left_armor_link">
+    <material>Gazebo/White</material>
+    <turnGravityOff>false</turnGravityOff>
+  </gazebo>
+  <gazebo reference="back_armor_link">
+    <material>Gazebo/White</material>
+    <turnGravityOff>false</turnGravityOff>
+  </gazebo>
+  <gazebo reference="front_armor_link">
+    <material>Gazebo/White</material>
     <turnGravityOff>false</turnGravityOff>
   </gazebo>

File: RoboRTS_Gazebo/robots/infantry.urdf.xacro (robot description, xacro)
@@ -685,5 +685,5 @@
       <geometry>
         <mesh
-          filename="package://roborts_gazebo/meshes/led_link.STL" />
+          filename="package://roborts_gazebo/meshes/led_link.STL" scale="0.001 0.001 0.001" />
       </geometry>
       <!-- <material
@@ -698,6 +698,6 @@
     type="fixed">
     <origin
-      xyz="0 0 0"
-      rpy="0 0 0" />
+      xyz="-0.094 0.2825 0.105"
+      rpy="0 3.1416 1.5708" />
     <parent
       link="base_link" />
@@ -707,3 +707,179 @@
       xyz="0 0 0" />
   </joint>
+  <link
+    name="front_armor_link">
+    <inertial>
+      <origin
+        xyz="-0.27282 -0.063339 0.010089"
+        rpy="0 0 0" />
+      <mass
+        value="0.028183" />
+      <inertia
+        ixx="0.00037048"
+        ixy="7.803E-06"
+        ixz="9.4378E-05"
+        iyy="0.0011379"
+        iyz="-1.4266E-06"
+        izz="0.0014674" />
+    </inertial>
+    <visual>
+      <origin
+        xyz="0.0 0.0 0.0"
+        rpy="0 0 0" />
+      <geometry>
+        <mesh
+          filename="package://roborts_gazebo/meshes/armor_basic.STL" scale="0.001 0.001 0.001"/>
+      </geometry>
+      <!-- <material
+        name="">
+        <color
+          rgba="1 0 0 1" />
+      </material> -->
+    </visual>
+  </link>
+  <joint
+    name="base_link_to_from_armor_joint"
+    type="fixed">
+    <origin
+      xyz="0.092 0.172 0.044"
+      rpy="0 3.1416 0" />
+    <parent
+      link="base_link" />
+    <child
+      link="front_armor_link" />
+    <axis
+      xyz="0 0 0" />
+  </joint>
+    <link
+    name="back_armor_link">
+    <inertial>
+      <origin
+        xyz="-0.27282 -0.063339 0.010089"
+        rpy="0 0 0" />
+      <mass
+        value="0.028183" />
+      <inertia
+        ixx="0.00037048"
+        ixy="7.803E-06"
+        ixz="9.4378E-05"
+        iyy="0.0011379"
+        iyz="-1.4266E-06"
+        izz="0.0014674" />
+    </inertial>
+    <visual>
+      <origin
+        xyz="0.0 0.0 0.0"
+        rpy="0 0 0" />
+      <geometry>
+        <mesh
+          filename="package://roborts_gazebo/meshes/armor_basic.STL" scale="0.001 0.001 0.001"/>
+      </geometry>
+      <!-- <material
+        name="">
+        <color
+          rgba="1 0 0 1" />
+      </material> -->
+    </visual>
+  </link>
+  <joint
+    name="base_link_to_back_armor_joint"
+    type="fixed">
+    <origin
+      xyz="-0.070 -0.172 0.044"
+      rpy="3.1416 0 0" />
+    <parent
+      link="base_link" />
+    <child
+      link="back_armor_link" />
+    <axis
+      xyz="0 0 0" />
+  </joint>
+  <link
+    name="left_armor_link">
+    <inertial>
+      <origin
+        xyz="-0.27282 -0.063339 0.010089"
+        rpy="0 0 0" />
+      <mass
+        value="0.028183" />
+      <inertia
+        ixx="0.00037048"
+        ixy="7.803E-06"
+        ixz="9.4378E-05"
+        iyy="0.0011379"
+        iyz="-1.4266E-06"
+        izz="0.0014674" />
+    </inertial>
+    <visual>
+      <origin
+        xyz="0.0 0.0 0.0"
+        rpy="0 0 0" />
+      <geometry>
+        <mesh
+          filename="package://roborts_gazebo/meshes/armor_basic.STL" scale="0.001 0.001 0.001"/>
+      </geometry>
+      <!-- <material
+        name="">
+        <color
+          rgba="1 0 0 1" />
+      </material> -->
+    </visual>
+  </link>
+  <joint
+    name="base_link_to_left_armor_joint"
+    type="fixed">
+    <origin
+      xyz="-0.157 -0.001 0.044"
+      rpy="3.1416 0 -1.5708" />
+    <parent
+      link="base_link" />
+    <child
+      link="left_armor_link" />
+    <axis
+      xyz="0 0 0" />
+  </joint>
+    <link
+    name="right_armor_link">
+    <inertial>
+      <origin
+        xyz="-0.27282 -0.063339 0.010089"
+        rpy="0 0 0" />
+      <mass
+        value="0.028183" />
+      <inertia
+        ixx="0.00037048"
+        ixy="7.803E-06"
+        ixz="9.4378E-05"
+        iyy="0.0011379"
+        iyz="-1.4266E-06"
+        izz="0.0014674" />
+    </inertial>
+    <visual>
+      <origin
+        xyz="0.0 0.0 0.0"
+        rpy="0 0 0" />
+      <geometry>
+        <mesh
+          filename="package://roborts_gazebo/meshes/armor_basic.STL" scale="0.001 0.001 0.001"/>
+      </geometry>
+      <!-- <material
+        name="">
+        <color
+          rgba="1 0 0 1" />
+      </material> -->
+    </visual>
+  </link>
+  <joint
+    name="base_link_to_right_armor_joint"
+    type="fixed">
+    <origin
+      xyz="0.1863 -0.001 0.044"
+      rpy="3.1416 0 1.5708" />
+    <parent
+      link="base_link" />
+    <child
+      link="right_armor_link" />
+    <axis
+      xyz="0 0 0" />
+  </joint>
 </robot>

Commit message: temporarily made the joint from yaw to pitch fixed so that the tf will be published without error; also changed the camera info which in turn added camera distortion to our simulation

File: RoboRTS_Gazebo/robots/infantry.gazebo.xacro (robot description, xacro)
@@ -165,8 +165,8 @@
       <update_rate>30.0</update_rate>
       <camera name="head">
-        <horizontal_fov>1.3962634</horizontal_fov>
+        <horizontal_fov>0.7280189</horizontal_fov>
         <image>
-          <width>1600</width>
-          <height>800</height>
+          <width>640</width>
+          <height>360</height>
           <format>R8G8B8</format>
         </image>
@@ -190,18 +190,18 @@
         <imageTopicName>image_raw</imageTopicName>
         <cameraInfoTopicName>camera_info</cameraInfoTopicName>
-        <frameName>camera_link_optical</frameName>
+        <frameName>camera_link</frameName>
         <!-- setting hackBaseline to anything but 0.0 will cause a misalignment
             between the gazebo sensor image and the frame it is supposed to
             be attached to -->
         <hackBaseline>0.0</hackBaseline>
-        <distortionK1>0.0</distortionK1>
-        <distortionK2>0.0</distortionK2>
+        <distortionK1>0.082613</distortionK1>
+        <distortionK2>0.043275</distortionK2>
         <distortionK3>0.0</distortionK3>
-        <distortionT1>0.0</distortionT1>
-        <distortionT2>0.0</distortionT2>
+        <distortionT1>-0.000823</distortionT1>
+        <distortionT2>0.002486</distortionT2>
         <CxPrime>0</CxPrime>
-        <Cx>0.0</Cx>
-        <Cy>0.0</Cy>
-        <focalLength>0.0</focalLength>
+        <Cx>340.780730</Cx>
+        <Cy>261.766523</Cy>
+        <focalLength>839.922884</focalLength>
       </plugin>
     </sensor>

File: RoboRTS_Gazebo/robots/infantry.transmission.xacro (robot description, xacro)
@@ -17,8 +17,8 @@
    <xacro:transmission_block joint_name="base_link_to_yaw_joint"/>
    <xacro:transmission_block joint_name="base_link_to_pitch_joint"/>
-   <xacro:transmission_block joint_name="base_link_to_fl_wheel_joint"/>
+   <!-- <xacro:transmission_block joint_name="base_link_to_fl_wheel_joint"/>
    <xacro:transmission_block joint_name="base_link_to_fr_wheel_joint"/>
    <xacro:transmission_block joint_name="base_link_to_bl_wheel_joint"/>
-   <xacro:transmission_block joint_name="base_link_to_br_wheel_joint"/>
+   <xacro:transmission_block joint_name="base_link_to_br_wheel_joint"/> -->
    <xacro:transmission_block joint_name="pitch_link_to_camera_wheel_joint"/>
 </robot>

File: RoboRTS_Gazebo/robots/infantry.urdf.xacro (robot description, xacro)
@@ -443,5 +443,5 @@
   <joint
     name="yaw_to_pitch_joint"
-    type="revolute">
+    type="fixed">
     <origin
       xyz="0 0 0.125"
@@ -453,9 +453,9 @@
     <axis
       xyz="0 1 0" />
-    <limit
+    <!-- <limit
       lower="-0.001"
       upper="0.001"
       effort="1000"
-      velocity="100" />
+      velocity="100" /> -->
   </joint>
   <link
@@ -491,5 +491,5 @@
       </material>
     </visual>
-    <collision>
+    <!-- <collision>
       <origin
         xyz="0 0 0"
@@ -499,5 +499,5 @@
           filename="package://roborts_gazebo/meshes/camera_link.STL" />
       </geometry>
-    </collision>
+    </collision> -->
   </link>
   <joint
@@ -739,5 +739,5 @@
   </link>
   <joint
-    name="base_link_to_from_armor_joint"
+    name="base_link_to_front_armor_joint"
     type="fixed">
     <origin

Commit message: modified camera features to match the reallife camera

File: RoboRTS_Gazebo/robots/infantry.gazebo.xacro (robot description, xacro)
@@ -165,8 +165,10 @@
       <update_rate>30.0</update_rate>
       <camera name="head">
-        <horizontal_fov>1.7280189</horizontal_fov>
+        <horizontal_fov>1.24256488</horizontal_fov>
         <image>
-          <width>640</width>
-          <height>360</height>
+          <!-- <width>640</width> -->
+          <!-- <height>360</height> -->
+          <width>1280</width>
+          <height>1024</height>
           <format>R8G8B8</format>
         </image>
@@ -201,7 +203,7 @@
         <distortionT2>0.002486</distortionT2>
         <CxPrime>0</CxPrime>
-        <Cx>0</Cx>
-        <Cy>0</Cy>
-        <focalLength>0</focalLength>
+        <Cx>640.5</Cx>
+        <Cy>512.5</Cy>
+        <focalLength>894.0460</focalLength>
       </plugin>
     </sensor>

File: RoboRTS_Gazebo/robots/infantry.urdf.xacro (robot description, xacro)
@@ -417,5 +417,5 @@
         izz="0.0037072" />
     </inertial>
-    <visual>
+    <!-- <visual>
       <origin
         xyz="0 0 0"
@@ -430,5 +430,5 @@
           rgba="1 1 1 1" />
       </material>
-    </visual>
+    </visual> -->
     <collision>
       <origin
@@ -503,7 +503,7 @@
   <joint
     name="pitch_link_to_camera_wheel_joint"
-    type="fixed">collision
-    <origin
-      xyz="0.041 0 0.049"
+    type="fixed">
+    <origin
+      xyz="0.128 0 -0.0492"
       rpy="0 0 0" />
     <parent
